File: Billy Bass Board/BillyBassBoard.brd (EAGLE design)
At the start: 60 x 70 mm, 106 parts, among them J1 MICRO-USB-AB, J10 MPT-2-SCREW, J11 MPT-2-SCREW, J2 MPT-2-SCREW, J3 MICRO-SD, J4 MPT-2-SCREW, J5 JST-XH-2, J6 3.5MM-JACK-4-TIP, J7 JST-XH-2, J8 MPT-2-SCREW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

Commit message: Updated files to match parts purchased
Parts:
- C12, C20, C21, C22, C23, C28, C3, C5, C7, C9: value 100nF ± 5% -> 0.1µF ± 5%
- C16: value 47nF ± 5% -> 0.047µF ± 10%
- R13: value 1kΩ ± 2% -> 1kΩ ± 1%
- R17: value 10Ω ± 2% -> 10Ω ± 1%
- R22, R23: value 2.4kΩ ± 2% -> 2.4kΩ ± 1%
- R27, R28, R29: value 330Ω ± 2% -> 330Ω ± 1%
